File: interface.kicad_sch (KiCad schematic)
At the start: 43 parts, among them J10 Conn_01x04_Socket, J11 Conn_01x04_Socket, J12 Conn_01x04_Socket, J13 Conn_01x04_Socket, J14 Conn_01x04_Socket, J15 Conn_01x04_Socket, J16 Conn_01x04_Socket, J17 Conn_01x04_Socket, J18 Conn_01x02_Socket, J19 Conn_01x02_Socket, J2 USB_C_Receptacle_USB2.0_16P, J20 Conn_01x02_Socket, J21 Conn_01x02_Socket, J22 Conn_01x02_Socket, J23 Conn_01x02_Socket, J24 Conn_01x02_Socket, J26 Conn_01x02_Socket, J27 Conn_01x02_Socket, J28 Conn_01x02_Socket, J29 Conn_01x03_Socket, J3 Conn_01x02_Socket, J4 Conn_01x02_Socket, J5 Conn_01x04_Socket, J6 Conn_01x08_Socket, J7 Conn_01x04_Socket, J8 Conn_01x04_Socket, J9 Conn_01x04_Socket, U4 ATA6561, U5 ATA6561

Commit message: test2
Parts:
- added J31: Conn_01x02_Socket, Connector_AMASS:AMASS_XT30PW-M_1x02_P2.50mm_Horizontal, symbol Connector:Conn_01x02_Socket
Changed lines of the file:
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@@
+	)
+	(symbol
+		(lib_id "Connector:Conn_01x02_Socket")
+		(at 111.76 52.07 0)
+		(unit 1)
+		(body_style 1)
+		(exclude_from_sim no)
+		(in_bom yes)
+		(on_board yes)
+		(in_pos_files yes)
+		(dnp no)
+		(fields_autoplaced yes)
+		(property "Reference" "J31"
+			(at 113.03 52.0699 0)
+			(show_name no)
+			(do_not_autoplace no)
+			(effects
+				(font
+					(size 1.27 1.27)
+				)
+				(justify left)
+			)
+		)
+		(property "Value" "Conn_01x02_Socket"
+			(at 113.03 54.6099 0)
+			(show_name no)
+			(do_not_autoplace no)
+			(effects
+				(font
+					(size 1.27 1.27)
+				)
+				(justify left)
+			)
+		)
+		(property "Footprint" "Connector_AMASS:AMASS_XT30PW-M_1x02_P2.50mm_Horizontal"
+			(at 111.76 52.07 0)
+			(hide yes)
+			(show_name no)
+			(do_not_autoplace no)
+			(effects
+				(font
+					(size 1.27 1.27)
+				)
+			)
+		)
+		(property "Datasheet" ""
+			(at 111.76 52.07 0)
+			(hide yes)
+			(show_name no)
+			(do_not_autoplace no)
+			(effects
+				(font
+					(size 1.27 1.27)
+				)
+			)
+		)
+		(property "Description" "Generic connector, single row, 01x02, script generated"
+			(at 111.76 52.07 0)
+			(hide yes)
+			(show_name no)
+			(do_not_autoplace no)
+			(effects
+				(font
+					(size 1.27 1.27)
+				)
+			)
+		)
+		(property "KLC_S3.3" ""
+			(at 111.76 52.07 0)
+			(hide yes)
+			(show_name no)
+			(do_not_autoplace no)
+			(effects
+				(font
+					(size 1.27 1.27)
+				)
+			)
+		)
+		(property "KLC_S4.1" ""
+			(at 111.76 52.07 0)
+			(hide yes)
+			(show_name no)
+			(do_not_autoplace no)
+			(effects
+				(font
+					(size 1.27 1.27)
+				)
+			)
+		)
+		(property "LCSC" ""
+			(at 111.76 52.07 0)
+			(hide yes)
+			(show_name no)
+			(do_not_autoplace no)
+			(effects
+				(font
+					(size 1.27 1.27)
+				)
+			)
+		)
+		(pin "1"
+		)
+		(pin "2"
+		)
+		(instances
+			(project "g474re_testboard_v1"
+				(path "/6701889f-a5e5-428d-8ee0-a9bdb287356c/a9436a45-4260-4b6f-9fed-953c709bebf7"
+					(reference "J31")
+					(unit 1)
+				)
+			)
+		)
 	)
 	(symbol
